Commit message: updated the code to work in gazebo classic

File: mr200_description/urdf/mr200.xacro (robot description, xacro)
@@ -151,5 +151,6 @@
   </inertial>
   <visual>
-    <origin xyz="0.001943 -0.001707 -0.298698" rpy="0 0 0"/>
+    <!-- <origin xyz="0.001943 -0.001707 -0.298698" rpy="0 0 0"/> -->
+    <origin xyz="0.001943 -0.001707 -0.228698" rpy="0 0 0"/>
     <geometry>
       <mesh filename="file://$(find mr200_description)/meshes/rplidar_1.stl" scale="0.001 0.001 0.001"/>
@@ -201,5 +202,6 @@
 </joint>
 <joint name="rplidar" type="fixed">
-  <origin xyz="-0.001943 0.001707 0.298698" rpy="0 0 0"/>
+  <!-- <origin xyz="-0.001943 0.001707 0.298698" rpy="0 0 0"/> -->
+  <origin xyz="-0.001943 0.001707 0.22" rpy="0 0 0"/>
   <parent link="base_link"/>
   <child link="rplidar_1"/>

Commit message: updated code for gazebo sim support

File: mr200_description/urdf/mr200.xacro (robot description, xacro)
@@ -4,4 +4,10 @@
 <xacro:include filename="$(find mr200_description)/urdf/mr200.trans" />
 <xacro:include filename="$(find mr200_description)/urdf/mr200.gazebo" />
+<link name="base_footprint"/>
+<joint name="base_joint" type="fixed">
+  <parent link="base_footprint"/>
+  <child link="base_link"/>
+  <origin xyz="0.0 0.0 0.0" rpy="0 0 0"/>
+</joint>
 <link name="base_link">
   <inertial>
@@ -165,27 +171,23 @@
   </collision>
 </link>
-<joint name="castor_rear_left" type="continuous">
+<joint name="castor_rear_left" type="fixed">
   <origin xyz="-0.202616 0.11528 0.091698" rpy="0 0 0"/>
   <parent link="base_link"/>
   <child link="castor_rear_left_1"/>
-  <axis xyz="-0.0 0.0 -1.0"/>
-</joint>
-<joint name="castor_rear_right" type="continuous">
+</joint>
+<joint name="castor_rear_right" type="fixed">
   <origin xyz="-0.202616 -0.11487 0.091698" rpy="0 0 0"/>
   <parent link="base_link"/>
   <child link="castor_rear_right_1"/>
-  <axis xyz="-0.0 -0.0 -1.0"/>
-</joint>
-<joint name="castor_front_left" type="continuous">
+</joint>
+<joint name="castor_front_left" type="fixed">
   <origin xyz="0.201234 0.11528 0.091698" rpy="0 0 0"/>
   <parent link="base_link"/>
   <child link="castor_front_left_1"/>
-  <axis xyz="-0.0 0.0 -1.0"/>
-</joint>
-<joint name="castor_front_right" type="continuous">
+</joint>
+<joint name="castor_front_right" type="fixed">
   <origin xyz="0.201234 -0.11487 0.091698" rpy="0 0 0"/>
   <parent link="base_link"/>
   <child link="castor_front_right_1"/>
-  <axis xyz="-0.0 -0.0 -1.0"/>
 </joint>
 <joint name="motor_right" type="continuous">
